Commit message: robot_vision package created to get the stream from camera

File: src/robot_description/urdf/robot.urdf.xacro (robot description, xacro)
@@ -1,153 +1,196 @@
 <?xml version="1.0"?>
 <robot xmlns:xacro="http://www.ros.org/wiki/xacro" name="my_robot">
-    <xacro:arg name="is_sim" default="true"/>
+    <xacro:arg name="is_sim" default="true" />
     <!-- Include gazebo parameters -->
-    <xacro:include filename="$(find robot_description)/urdf/robot_gazebo.xacro"/>
+    <xacro:include filename="$(find robot_description)/urdf/robot_gazebo.xacro" />
     <!-- <xacro:include filename="$(find robot_description)/urdf/common_properties.xacro"/> -->
     <!-- <xacro:include filename="$(find robot_description)/urdf/camera.xacro"/> -->
     <!-- ROS2 control -->
-    <xacro:include filename="$(find robot_description)/urdf/robot_ros2_control.xacro"/>
-    <link name="base_footprint"/>
+    <xacro:include filename="$(find robot_description)/urdf/robot_ros2_control.xacro" />
+    <link name="base_footprint" />
     <link name="base_link">
         <inertial>
-            <origin xyz="0.0 0.0 0.04" rpy="0.0 0.25 0.3"/>
-            <mass value="8.2573504e-01"/>
+            <origin xyz="0.0 0.0 0.04" rpy="0.0 0.25 0.3" />
+            <mass value="8.2573504e-01" />
             <inertia ixx="2.2124416e-02" ixy="-1.2294101e-04" ixz="3.4938785e-04"
-                     iyy="2.1193702e-02" iyz="-5.0120904e-05"
-                     izz="2.0064271e-02"/>
+                iyy="2.1193702e-02" iyz="-5.0120904e-05"
+                izz="2.0064271e-02" />
         </inertial>
         <visual>
-            <origin rpy="0 0 0" xyz = "0 0 0"/>
+            <origin rpy="0 0 0" xyz="0 0 0" />
             <geometry>
-                <!-- <mesh filename="package://robot_description/meshes/base_link.STL" scale="1 1 1"/> -->
-                <mesh filename="file://$(find robot_description)/meshes/base_link.STL"/>
+                <!-- <mesh filename="package://robot_description/meshes/base_link.STL" scale="1 1
+                1"/> -->
+                <mesh filename="file://$(find robot_description)/meshes/base_link.STL" />
             </geometry>
         </visual>
         <collision>
-            <origin rpy="0 0 0" xyz = "0 0 0"/>
+            <origin rpy="0 0 0" xyz="0 0 0" />
             <geometry>
-                <!-- <mesh filename="package://robot_description/meshes/base_link.STL" scale="1 1 1"/> -->
-                <mesh filename="file://$(find robot_description)/meshes/base_link.STL"/>
+                <!-- <mesh filename="package://robot_description/meshes/base_link.STL" scale="1 1
+                1"/> -->
+                <mesh filename="file://$(find robot_description)/meshes/base_link.STL" />
             </geometry>
         </collision>
     </link>
     <joint name="base_joint" type="fixed">
-        <parent link="base_footprint"/>
-        <child link="base_link"/>
-        <origin rpy="0 0 0 " xyz="0 0 0.033"/>
+        <parent link="base_footprint" />
+        <child link="base_link" />
+        <origin rpy="0 0 0 " xyz="0 0 0.033" />
     </joint>
     <!-- right wheel link and joint -->
     <link name="wheel_right_link">
         <inertial>
-            <origin xyz="0 -0.014 0" rpy="0.0 0.0 0.0"/>
-            <mass value="0.0530086090966721"/>
-            <inertia ixx="1.88176298336665e-05" ixy="-4.8444933029987e-10" ixz="1.55163708851143e-08"
-                     iyy="3.11510738647764e-05" iyz="-6.93560663069607e-11"
-                     izz="1.8801969558182e-05"/>
+            <origin xyz="0 -0.014 0" rpy="0.0 0.0 0.0" />
+            <mass value="0.0530086090966721" />
+            <inertia ixx="1.88176298336665e-05" ixy="-4.8444933029987e-10"
+                ixz="1.55163708851143e-08"
+                iyy="3.11510738647764e-05" iyz="-6.93560663069607e-11"
+                izz="1.8801969558182e-05" />
         </inertial>
-        <visual >
-            <origin xyz="0 0.0 0.0" rpy="1.57 0.0 0.0"/>
+        <visual>
+            <origin xyz="0 0.0 0.0" rpy="1.57 0.0 0.0" />
             <geometry>
-                <!-- <mesh filename="package://robot_description/meshes/wheel_right_link.STL" scale="1 1 1"/> -->
-                <mesh filename="file://$(find robot_description)/meshes/wheel_right_link.STL"/>
+                <!-- <mesh filename="package://robot_description/meshes/wheel_right_link.STL"
+                scale="1 1 1"/> -->
+                <mesh filename="file://$(find robot_description)/meshes/wheel_right_link.STL" />
             </geometry>
         </visual>
         <collision>
-            <origin xyz="0.0 -0.015 0.0" rpy="1.57 0.0 0.0"/>
+            <origin xyz="0.0 -0.015 0.0" rpy="1.57 0.0 0.0" />
             <geometry>
-                <sphere radius="0.033"/>
+                <sphere radius="0.033" />
             </geometry>
         </collision>
     </link>
     <joint name="wheel_right_joint" type="continuous">
-        <parent link="base_link"/>
-        <child link="wheel_right_link"/>
-        <origin xyz="0.0 -0.07 0.0" rpy="0.0 0.0 0.0"/>
-        <axis xyz="0.0 1 0.0"/>
+        <parent link="base_link" />
+        <child link="wheel_right_link" />
+        <origin xyz="0.0 -0.07 0.0" rpy="0.0 0.0 0.0" />
+        <axis xyz="0.0 1 0.0" />
     </joint>
     <!-- left wheel link and joint -->
     <link name="wheel_left_link">
         <inertial>
-            <origin xyz="0.0 0.014 0.0" rpy="0.0 0.0 0.0"/>
-            <mass value="0.0530086043217644"/>
-            <inertia ixx="1.8792911368909e-05" ixy="3.31256392204584e-10" ixz="-1.14082001665767e-08"
-                    iyy="3.11510738759073e-05" iyz="-3.60499245082192e-10"
-                    izz="1.88266886146847e-05"/>
+            <origin xyz="0.0 0.014 0.0" rpy="0.0 0.0 0.0" />
+            <mass value="0.0530086043217644" />
+            <inertia ixx="1.8792911368909e-05" ixy="3.31256392204584e-10"
+                ixz="-1.14082001665767e-08"
+                iyy="3.11510738759073e-05" iyz="-3.60499245082192e-10"
+                izz="1.88266886146847e-05" />
         </inertial>
-        <visual >
-            <origin xyz="0 0.0 0.0" rpy="-1.57 0.0 0.0"/>
+        <visual>
+            <origin xyz="0 0.0 0.0" rpy="-1.57 0.0 0.0" />
             <geometry>
-                <!-- <mesh filename="package://robot_description/meshes/wheel_left_link.STL" scale="1 1 1"/> -->
-                <mesh filename="file://$(find robot_description)/meshes/wheel_left_link.STL"/>
+                <!-- <mesh filename="package://robot_description/meshes/wheel_left_link.STL"
+                scale="1 1 1"/> -->
+                <mesh filename="file://$(find robot_description)/meshes/wheel_left_link.STL" />
             </geometry>
         </visual>
         <collision>
-            <origin xyz="0.0 0.015 0.0" rpy="1.57 0.0 0.0"/>
+            <origin xyz="0.0 0.015 0.0" rpy="1.57 0.0 0.0" />
             <geometry>
-                <sphere radius="0.033"/>
+                <sphere radius="0.033" />
             </geometry>
         </collision>
     </link>
     <joint name="wheel_left_joint" type="continuous">
-        <parent link="base_link"/>
-        <child link="wheel_left_link"/>
-        <origin xyz="0.0 0.07 0.0" rpy="0.0 0.0 0.0"/>
-        <axis xyz="0.0 1 0.0"/>
+        <parent link="base_link" />
+        <child link="wheel_left_link" />
+        <origin xyz="0.0 0.07 0.0" rpy="0.0 0.0 0.0" />
+        <axis xyz="0.0 1 0.0" />
     </joint>
     <!-- caster wheel front link -->
     <link name="caster_front_link">
-       <inertial>
-        <origin xyz="3.89968128948481e-07 2.40073004698083e-07 0.00219173397061506" rpy="0.0 0.0 0.0"/>
-        <mass value="1.44379565037903e-06"/>
-        <inertia ixx="7.23075276010246e-11" ixy="-6.10956883467859e-16" ixz="2.22849693525031e-15"
-                 iyy="3.8713793085917e-11" iyz="2.93909858781952e-15"
-                 izz="1.00967486676306e-10"/>
-       </inertial>
-       <visual>
-           <origin xyz="0.0 0.0 0.0" rpy="0.0 0.0 0.0"/>
-           <geometry>
-               <!-- <mesh filename="package://robot_description/meshes/caster_front_link.STL" scale="1 1 1"/> -->
-                <mesh filename="file://$(find robot_description)/meshes/caster_front_link.STL"/>
+        <inertial>
+            <origin xyz="3.89968128948481e-07 2.40073004698083e-07 0.00219173397061506"
+                rpy="0.0 0.0 0.0" />
+            <mass value="1.44379565037903e-06" />
+            <inertia ixx="7.23075276010246e-11" ixy="-6.10956883467859e-16"
+                ixz="2.22849693525031e-15"
+                iyy="3.8713793085917e-11" iyz="2.93909858781952e-15"
+                izz="1.00967486676306e-10" />
+        </inertial>
+        <visual>
+            <origin xyz="0.0 0.0 0.0" rpy="0.0 0.0 0.0" />
+            <geometry>
+                <!-- <mesh filename="package://robot_description/meshes/caster_front_link.STL"
+                scale="1 1 1"/> -->
+                <mesh filename="file://$(find robot_description)/meshes/caster_front_link.STL" />
             </geometry>
         </visual>
         <collision>
-            <origin xyz="0.0 0.0 0.0" rpy="0.0 0.0 0.0"/>
+            <origin xyz="0.0 0.0 0.0" rpy="0.0 0.0 0.0" />
             <geometry>
-                <sphere radius="0.005"/>
+                <sphere radius="0.005" />
             </geometry>
         </collision>
     </link>
     <joint name="caster_front_joint" type="fixed">
-        <parent link="base_link"/>
-        <child link="caster_front_link"/>
-        <origin xyz="0.04755 0 -0.0275" rpy="0.0 0.0 0.0"/>
+        <parent link="base_link" />
+        <child link="caster_front_link" />
+        <origin xyz="0.04755 0 -0.0275" rpy="0.0 0.0 0.0" />
     </joint>
     <!-- caster wheel rear link -->
     <link name="caster_rear_link">
         <inertial>
-            <origin xyz="3.8996812895542e-07 2.40073004698083e-07 0.00219173397061509" rpy="0.0 0.0 0.0"/>
-            <mass value="1.44379265037902e-06"/>
-            <inertia ixx="7.23075276010246e-11" ixy="-6.10956872363424e-16" ixz="2.22849693527207e-15"
-                    iyy="3.89137930859167e-11" iyz="2.939098587861e-15"
-                    izz="1.00967486676306e-10"/>
+            <origin xyz="3.8996812895542e-07 2.40073004698083e-07 0.00219173397061509"
+                rpy="0.0 0.0 0.0" />
+            <mass value="1.44379265037902e-06" />
+            <inertia ixx="7.23075276010246e-11" ixy="-6.10956872363424e-16"
+                ixz="2.22849693527207e-15"
+                iyy="3.89137930859167e-11" iyz="2.939098587861e-15"
+                izz="1.00967486676306e-10" />
         </inertial>
         <visual>
-            <origin xyz="0.0 0.0 0.0" rpy="0.0 0.0 0.0"/>
+            <origin xyz="0.0 0.0 0.0" rpy="0.0 0.0 0.0" />
             <geometry>
-                <!-- <mesh filename="package://robot_description/meshes/caster_rear_link.STL" scale="1 1 1"/> -->
-                <mesh filename="file://$(find robot_description)/meshes/caster_rear_link.STL"/>
+                <!-- <mesh filename="package://robot_description/meshes/caster_rear_link.STL"
+                scale="1 1 1"/> -->
+                <mesh filename="file://$(find robot_description)/meshes/caster_rear_link.STL" />
             </geometry>
         </visual>
         <collision>
-            <origin xyz="0.0 0.0 0.0" rpy="0.0 0.0 0.0"/>
+            <origin xyz="0.0 0.0 0.0" rpy="0.0 0.0 0.0" />
             <geometry>
-                <sphere radius="0.005"/>
+                <sphere radius="0.005" />
             </geometry>
         </collision>
     </link>
     <joint name="caster_rear_joint" type="fixed">
-        <parent link="base_link"/>
-        <child link="caster_rear_link"/>
-        <origin xyz="-0.04755 0 -0.0275" rpy="0.0 0.0 0.0"/>
+        <parent link="base_link" />
+        <child link="caster_rear_link" />
+        <origin xyz="-0.04755 0 -0.0275" rpy="0.0 0.0 0.0" />
+    </joint>
+    <link name="imu_link">
+        <inertial>
+            <origin xyz="-0.00552433659106688 0.000168210391520346 0.000514000497342681" rpy="0 0 0" />
+            <mass value="0.000528415362211671" />
+            <inertia ixx="1.46176048428261E-08" ixy="1.40015117949421E-10"
+                ixz="-1.99633872937403E-12"
+                iyy="8.59662482954888E-09" iyz="7.52375112767959E-12"
+                izz="2.30279421279312E-08" />
+        </inertial>
+        <visual>
+            <origin xyz="0 0 0" rpy="0 0 0" />
+            <geometry>
+                <mesh filename="package://robot_description/meshes/imu_link.STL" />
+            </geometry>
+            <material name="">
+                <color rgba="0.792156862745098 0.819607843137255 0.933333333333333 1" />
+            </material>
+        </visual>
+        <collision>
+            <origin xyz="0 0 0" rpy="0 0 0" />
+            <geometry>
+                <mesh filename="package://robot_description/meshes/imu_link.STL" />
+            </geometry>
+        </collision>
+    </link>
+    <joint name="imu_joint" type="fixed">
+        <origin xyz="0 0 0.0698986241758014" rpy="0 0 0" />
+        <parent link="base_link" />
+        <child link="imu_link" />
+        <axis xyz="0 0 0" />
     </joint>
 </robot>

File: src/robot_description/urdf/robot_gazebo.xacro (robot description, xacro)
@@ -35,7 +35,7 @@
         <maxvel>0.1</maxvel>
     </gazebo> -->
-    <gazebo reference="base_link">
+    <!-- <gazebo reference="base_link">
         <material>Gazebo/White</material>
-    </gazebo>
+    </gazebo> -->
      <gazebo reference="wheel_right_link">
         <mu1>1.0</mu1>
@@ -73,8 +73,64 @@
     </gazebo>
     <gazebo>
-        <plugin filename="libgazebo_ros2_control.so" name="gazebo_ros2_control">
+        <!-- <plugin filename="libgazebo_ros2_control.so" name="gazebo_ros2_control">
             <parameters>$(find robot_controller)/config/robot_controllers.yaml</parameters>
-            <!-- <robot_param>robot_description</robot_param> -->
-        </plugin>
+            <robot_param>robot_description</robot_param>
+        </plugin> -->
+        <plugin filename="ign_ros2_control-system" name="ign_ros2_control::IgnitionROS2ControlPlugin">
+        <parameters>$(find robot_controller)/config/robot_controllers.yaml</parameters>
+      </plugin>
+      <plugin filename="ignition-gazebo-imu-system" name="ignition::gazebo::systems::Imu">
+      </plugin>
     </gazebo>
+    <!-- IMU -->
+    <gazebo reference="imu_link">
+        <sensor name="imu" type="imu">
+            <always_on>true</always_on>
+            <update_rate>100</update_rate>
+            <gz_frame_id>imu_link</gz_frame_id>
+            <topic>imu</topic>
+            <imu>
+            <angular_velocity>
+                <x>
+                <noise type="gaussian">
+                    <mean>0.0</mean>
+                    <stddev>2e-4</stddev>
+                </noise>
+                </x>
+                <y>
+                <noise type="gaussian">
+                    <mean>0.0</mean>
+                    <stddev>2e-4</stddev>
+                </noise>
+                </y>
+                <z>
+                <noise type="gaussian">
+                    <mean>0.0</mean>
+                    <stddev>2e-4</stddev>
+                </noise>
+                </z>
+            </angular_velocity>
+            <linear_acceleration>
+                <x>
+                <noise type="gaussian">
+                    <mean>0.0</mean>
+                    <stddev>1.7e-2</stddev>
+                </noise>
+                </x>
+                <y>
+                <noise type="gaussian">
+                    <mean>0.0</mean>
+                    <stddev>1.7e-2</stddev>
+                </noise>
+                </y>
+                <z>
+                <noise type="gaussian">
+                    <mean>0.0</mean>
+                    <stddev>1.7e-2</stddev>
+                </noise>
+                </z>
+            </linear_acceleration>
+            </imu>
+        </sensor>
+  </gazebo>
 </robot>

File: src/robot_description/urdf/robot_ros2_control.xacro (robot description, xacro)
@@ -5,5 +5,6 @@
         <xacro:if value="$(arg is_sim)">
             <hardware>
-                <plugin>gazebo_ros2_control/GazeboSystem</plugin>
+                <!-- <plugin>gazebo_ros2_control/GazeboSystem</plugin> -->
+                <plugin>ign_ros2_control/IgnitionSystem</plugin>
             </hardware>
         </xacro:if>

Commit message: implemented line following robot code and modified wheel radius and wheel separation values in controllers.yaml , controller.launch.py, robot.urdf.xacro files

File: src/robot_description/urdf/robot.urdf.xacro (robot description, xacro)
@@ -37,5 +37,5 @@
         <parent link="base_footprint" />
         <child link="base_link" />
-        <origin rpy="0 0 0 " xyz="0 0 0.033" />
+        <origin rpy="0 0 0 " xyz="0 0 0.0335" />
     </joint>
     <!-- right wheel link and joint -->
@@ -60,5 +60,5 @@
             <origin xyz="0.0 -0.015 0.0" rpy="1.57 0.0 0.0" />
             <geometry>
-                <sphere radius="0.033" />
+                <sphere radius="0.0335" />
             </geometry>
         </collision>
@@ -91,5 +91,5 @@
             <origin xyz="0.0 0.015 0.0" rpy="1.57 0.0 0.0" />
             <geometry>
-                <sphere radius="0.033" />
+                <sphere radius="0.0335" />
             </geometry>
         </collision>
